File: Main-Board.brd (EAGLE design)
At the start: 160 x 100 mm, 13 parts, among them IC1 Z80CPU, IC4 XR-16C550P, IC5 HM62256DIP, J1 DCJ0202

Commit message: Add Readme, Add Wait line for IO
Connections:
- new net WAIT: IC1.24, SV2.27
- net VCC: no longer IC1.24
Changed lines of the file:
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@@
 <contactref element="R1" pad="2"/>
 <contactref element="IC1" pad="25"/>
-<contactref element="IC1" pad="24"/>
 <contactref element="IC1" pad="16"/>
 <contactref element="IC1" pad="17"/>
@@
 <wire x1="-33.02" y1="22.86" x2="-35.56" y2="22.86" width="0" layer="19" extent="1-1"/>
 <wire x1="-25.4" y1="17.78" x2="-33.02" y2="22.86" width="0" layer="19" extent="1-1"/>
-<wire x1="-22.86" y1="17.78" x2="-25.4" y2="17.78" width="0" layer="19" extent="1-1"/>
 <wire x1="-25.4" y1="2.54" x2="-25.4" y2="17.78" width="0" layer="19" extent="1-1"/>
 <wire x1="-22.86" y1="2.54" x2="-25.4" y2="2.54" width="0" layer="19" extent="1-1"/>
@@
 <wire x1="-38.1" y1="83.82" x2="-27.94" y2="83.82" width="0" layer="19" extent="1-1"/>
 </signal>
+<signal name="WAIT">
+<contactref element="IC1" pad="24"/>
+<contactref element="SV2" pad="27"/>
+<wire x1="-22.86" y1="17.78" x2="-30.48" y2="97.79" width="0" layer="19" extent="1-1"/>
+</signal>
 </signals>
