File: Main-Board.sch (EAGLE design)
At the start: 13 parts, among them IC1 Z80CPU, IC4 XR-16C550P, IC5 HM62256DIP, J1 DCJ0202

Commit message: Add Readme, Add Wait line for IO
Connections:
- new net WAIT: IC1.WAIT, SV2.27
- net VCC: no longer IC1.WAIT
Changed lines of the file:
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@@
 <wire x1="-5.08" y1="45.72" x2="-25.4" y2="45.72" width="0.1524" layer="91"/>
 <wire x1="-25.4" y1="45.72" x2="-25.4" y2="55.88" width="0.1524" layer="91"/>
-<pinref part="IC1" gate="1" pin="WAIT"/>
 <wire x1="-25.4" y1="55.88" x2="-25.4" y2="58.42" width="0.1524" layer="91"/>
-<wire x1="-25.4" y1="58.42" x2="-25.4" y2="66.04" width="0.1524" layer="91"/>
-<wire x1="-25.4" y1="66.04" x2="-25.4" y2="68.58" width="0.1524" layer="91"/>
-<wire x1="-5.08" y1="63.5" x2="-7.62" y2="63.5" width="0.1524" layer="91"/>
-<wire x1="-7.62" y1="63.5" x2="-7.62" y2="66.04" width="0.1524" layer="91"/>
-<wire x1="-7.62" y1="66.04" x2="-25.4" y2="66.04" width="0.1524" layer="91"/>
-<junction x="-25.4" y="66.04"/>
+<wire x1="-25.4" y1="58.42" x2="-25.4" y2="68.58" width="0.1524" layer="91"/>
 <pinref part="IC1" gate="1" pin="INT"/>
 <wire x1="-5.08" y1="58.42" x2="-25.4" y2="58.42" width="0.1524" layer="91"/>
@@
 </segment>
 </net>
+<net name="WAIT" class="0">
+<segment>
+<pinref part="IC1" gate="1" pin="WAIT"/>
+<wire x1="-5.08" y1="63.5" x2="-7.62" y2="63.5" width="0.1524" layer="91"/>
+<wire x1="-7.62" y1="63.5" x2="-7.62" y2="-7.62" width="0.1524" layer="91"/>
+<wire x1="-7.62" y1="-7.62" x2="317.5" y2="-7.62" width="0.1524" layer="91"/>
+<wire x1="317.5" y1="-7.62" x2="317.5" y2="45.72" width="0.1524" layer="91"/>
+<pinref part="SV2" gate="G$1" pin="27"/>
+<wire x1="317.5" y1="45.72" x2="322.58" y2="45.72" width="0.1524" layer="91"/>
+<label x="317.5" y="45.72" size="1.778" layer="95"/>
+</segment>
+</net>
