File: PS2.brd (EAGLE design)
At the start: 106.7 x 26.3 mm, 11 parts, among them IC1 ATMEGA328-20P

Commit message: Reposition Capacitor
Parts:
- moved C4 5.08 mm to (27.9, 8.89), turned to 0 degrees
Changed lines of the file:
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@@
 <attribute name="MPN" value="" x="-3.81" y="15.24" size="1.778" layer="27" rot="R270" display="off"/>
 </element>
-<element name="C4" library="capacitor-wima" package="C5B3" value="0.1µ" x="22.86" y="8.89" rot="R180"/>
+<element name="C4" library="capacitor-wima" package="C5B3" value="0.1µ" x="27.94" y="8.89"/>
 <element name="C5" library="capacitor-wima" package="C5B3" value="0.1µ" x="102.87" y="12.7" rot="R90"/>
 </elements>
