File: VideoAudio.sch (EAGLE design)
At the start: 33 parts, among them IC1 MAX734CPA, IC2 MAX660CPA, IC3 TMS9918A, Q1 10.738635MHz, T1 2N3904, X1 TOBU3

Commit message: Add Audio and Video to videoboard, not yet ready
Parts:
- added C11, C12, C13, C14, C15, C16, C17, C18, C19, C20, C21, C22, C23, C24, C25, C26: 10µF, rcl:C-EU050-025X075
- added QG1: 2MHz, crystal:XO-14
- added SV1, SV2: (no value), con-lstb:MA10-1
- added U1: AY-3-8912, oldchips:AY-3-8912
- added V3: 74238N, 74ttl-din:74238N
- added V4: 7432N, 74ttl-din:7432N
- added X2: TOBU3, con-hirschmann:TOBU3
Connections:
- new net !RESET: IC3.SYNC/!RESET, JP1.!RESET, U1>NAME./RESET
- new net A0: V31.C
- new net N$11: V31.Y6, V4/1.B
- new net N$15: U1>NAME.BC1, V4/1.Y
- new net N$16: V31.Y1, V4/1.A, V4/2.A
- new net N$17: U1>NAME.BDIR, V4/2.Y
- new net N$18: V31.Y5, V4/2.B
- new net N$19: SV1.1, U1>NAME.IOB0
- new net N$20: SV1.2, U1>NAME.IOB1
- new net N$21: SV1.3, U1>NAME.IOB2
- new net N$22: SV1.4, U1>NAME.IOB3
- new net N$23: SV1.5, U1>NAME.IOB4
- new net N$24: SV1.6, U1>NAME.IOB5
- new net N$25: SV1.7, U1>NAME.IOB6
- new net N$26: SV1.8, U1>NAME.IOB7
- new net N$27: QG1.OUT, U1>NAME.CLOCK
- new net N$28: SV2.1, U1>NAME.IOA0
- new net N$29: SV2.2, U1>NAME.IOA1
- new net N$30: SV2.3, U1>NAME.IOA2
- new net N$31: SV2.4, U1>NAME.IOA3
- new net N$32: SV2.5, U1>NAME.IOA4
- new net N$33: SV2.6, U1>NAME.IOA5
- new net N$34: SV2.7, U1>NAME.IOA6
- new net N$35: SV2.8, U1>NAME.IOA7
- net !AUDIOEN: now also V31.!G2B
- net !RD: now also V31.A
- net !WR: now also V31.B
- net D0: now also U1>NAME.DA0
- net D1: now also U1>NAME.DA1
- net D2: now also U1>NAME.DA2
- net D3: now also U1>NAME.DA3
- net D4: now also U1>NAME.DA4
- net D5: now also U1>NAME.DA5
- net D6: now also U1>NAME.DA6
- net D7: now also U1>NAME.DA7
- net GND: now also QG1.GND, SV1.10, SV2.10, U1P.GND, V3/-UB.-UB, V31.!G2A, V4/-UB.-UB, X2.2
- net N$6: now also U1>NAME.A_CHA, U1>NAME.A_CHB, U1>NAME.A_CHC, X2.1; no longer IC3.SYNC/!RESET, JP1.!RESET
- net VCC: now also C11.1, C12.1, C13.1, C14.1, C15.1, C16.1, C17.1, C18.1, C19.1, C20.1, C21.1, C22.1, C23.1, C24.1, C25.1, C26.1, QG1.VCC, SV1.9, SV2.9, U1>NAME.BC2, U1P.VCC, V3/+UB.+UB, V31.G1, V4/+UB.+UB
Other:
- note added: "A0 = 0: Address Write A0 = 1: Data Write / Read"
