File: Muddi.sch (EAGLE design)
At the start: 15 parts, among them IC1 7805TV, J1 DCJ0202

Commit message: Add more Texts
Connections:
- net N$1 renamed D0
- net N$24 renamed A15
- net N$37 renamed !BUSACK
- net N$38 renamed !BUSREQ
- net N$39 renamed !M1
- net N$40 renamed !RESE
- net N$41 renamed !HALT
- net N$42 renamed !NMI
- net N$43 renamed !INT
- net N$44 renamed CLK
- net N$45 renamed !MREQ
- net N$46 renamed !IOREQ
- net N$47 renamed !WAIT
- net N$48 renamed !RD
- net N$49 renamed !WR
- net N$8 renamed D7
- net N$9 renamed A0
Changed lines of the file:
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@@
 </busses>
 <nets>
-<net name="N$1" class="0">
+<net name="D0" class="0">
 <segment>
 <pinref part="JP1" gate="A" pin="D0"/>
@@
 </segment>
 </net>
-<net name="N$8" class="0">
+<net name="D7" class="0">
 <segment>
 <pinref part="JP6" gate="A" pin="D7"/>
@@
 </segment>
 </net>
-<net name="N$9" class="0">
+<net name="A0" class="0">
 <segment>
 <pinref part="JP1" gate="A" pin="A0"/>
@@
 </segment>
 </net>
-<net name="N$24" class="0">
+<net name="A15" class="0">
 <segment>
 <pinref part="JP2" gate="A" pin="A15"/>
@@
 </segment>
 </net>
-<net name="N$37" class="0">
+<net name="!BUSACK" class="0">
 <segment>
 <pinref part="JP2" gate="A" pin="!BUSACK"/>
@@
 </segment>
 </net>
-<net name="N$38" class="0">
+<net name="!BUSREQ" class="0">
 <segment>
 <pinref part="JP1" gate="A" pin="!BUSRQ"/>
@@
 </segment>
 </net>
-<net name="N$39" class="0">
+<net name="!M1" class="0">
 <segment>
 <pinref part="JP2" gate="A" pin="!M1"/>
@@
 </segment>
 </net>
-<net name="N$40" class="0">
+<net name="!RESE" class="0">
 <segment>
 <pinref part="JP1" gate="A" pin="!RESET"/>
@@
 </segment>
 </net>
-<net name="N$41" class="0">
+<net name="!HALT" class="0">
 <segment>
 <pinref part="JP2" gate="A" pin="!HALT"/>
@@
 </segment>
 </net>
-<net name="N$42" class="0">
+<net name="!NMI" class="0">
 <segment>
 <pinref part="JP1" gate="A" pin="!NMI"/>
@@
 </segment>
 </net>
-<net name="N$43" class="0">
+<net name="!INT" class="0">
 <segment>
 <pinref part="JP2" gate="A" pin="!INT"/>
@@
 </segment>
 </net>
-<net name="N$44" class="0">
+<net name="CLK" class="0">
 <segment>
 <pinref part="JP1" gate="A" pin="CLK"/>
@@
 </segment>
 </net>
-<net name="N$45" class="0">
+<net name="!MREQ" class="0">
 <segment>
 <pinref part="JP2" gate="A" pin="!MREQ"/>
@@
 </segment>
 </net>
-<net name="N$46" class="0">
+<net name="!IOREQ" class="0">
 <segment>
 <pinref part="JP1" gate="A" pin="!IOREQ"/>
@@
 </segment>
 </net>
-<net name="N$47" class="0">
+<net name="!WAIT" class="0">
 <segment>
 <pinref part="JP2" gate="A" pin="!WAIT"/>
@@
 </segment>
 </net>
-<net name="N$48" class="0">
+<net name="!RD" class="0">
 <segment>
 <pinref part="JP1" gate="A" pin="!RD"/>
@@
 </segment>
 </net>
-<net name="N$49" class="0">
+<net name="!WR" class="0">
 <segment>
 <pinref part="JP2" gate="A" pin="!WR"/>

Commit message: Fix stupid VCC/GND mistakes on Address decoder
Connections:
- removed net N$28: D1.A, J1.1
- new net N$1: D1.A, J1.3
- net GND: now also J1.1; no longer J1.3
Other:
- moved on the sheet: J1
Changed lines of the file:
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@@
 <instance part="JP5" gate="A" x="137.16" y="172.72"/>
 <instance part="JP6" gate="A" x="175.26" y="172.72"/>
-<instance part="J1" gate="G$1" x="-43.18" y="254"/>
+<instance part="J1" gate="G$1" x="-33.02" y="254" rot="R180"/>
 <instance part="GND" gate="1" x="12.7" y="241.3"/>
 <instance part="VCC" gate="VCC" x="12.7" y="266.7"/>
@@
 <instance part="P+1" gate="VCC" x="-12.7" y="279.4"/>
 <instance part="GND1" gate="1" x="-25.4" y="261.62"/>
-<instance part="GND3" gate="1" x="-30.48" y="241.3"/>
+<instance part="GND3" gate="1" x="-40.64" y="241.3"/>
 <instance part="MAX811" gate="G$1" x="-38.1" y="134.62"/>
 <instance part="GND4" gate="1" x="-43.18" y="121.92"/>
@@
 </segment>
 <segment>
-<pinref part="J1" gate="G$1" pin="3"/>
 <pinref part="GND3" gate="1" pin="GND"/>
-<wire x1="-35.56" y1="251.46" x2="-30.48" y2="251.46" width="0.1524" layer="91"/>
-<wire x1="-30.48" y1="251.46" x2="-30.48" y2="243.84" width="0.1524" layer="91"/>
 <pinref part="C2" gate="G$1" pin="-"/>
 <wire x1="-45.72" y1="261.62" x2="-53.34" y2="261.62" width="0.1524" layer="91"/>
 <wire x1="-53.34" y1="261.62" x2="-53.34" y2="243.84" width="0.1524" layer="91"/>
-<wire x1="-53.34" y1="243.84" x2="-30.48" y2="243.84" width="0.1524" layer="91"/>
-<junction x="-30.48" y="243.84"/>
+<wire x1="-53.34" y1="243.84" x2="-40.64" y2="243.84" width="0.1524" layer="91"/>
+<pinref part="J1" gate="G$1" pin="1"/>
+<wire x1="-40.64" y1="251.46" x2="-40.64" y2="243.84" width="0.1524" layer="91"/>
+<junction x="-40.64" y="243.84"/>
 </segment>
 <segment>
@@
 </segment>
 </net>
-<net name="N$28" class="0">
-<segment>
-<pinref part="J1" gate="G$1" pin="1"/>
+<net name="N$1" class="0">
+<segment>
+<pinref part="J1" gate="G$1" pin="3"/>
+<wire x1="-40.64" y1="256.54" x2="-40.64" y2="261.62" width="0.1524" layer="91"/>
+<wire x1="-40.64" y1="261.62" x2="-35.56" y2="261.62" width="0.1524" layer="91"/>
 <pinref part="D1" gate="1" pin="A"/>
-<wire x1="-35.56" y1="256.54" x2="-35.56" y2="264.16" width="0.1524" layer="91"/>
-</segment>
-</net>
+<wire x1="-35.56" y1="261.62" x2="-35.56" y2="264.16" width="0.1524" layer="91"/>
+</segment>
+</net>
