File: CPU.brd (EAGLE design)
At the start: 106.7 x 34 mm, 11 parts, among them IC1 Z80CPU

Commit message: Fix Routing Issues with PowerPlanes
Routing:
- net VCC: track 0.00 -> 8.22 mm, vias 0 -> 4
Changed lines of the file:
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@@
 <contactref element="JP1" pad="53"/>
 <contactref element="R1" pad="1"/>
-<wire x1="35.56" y1="6.35" x2="38.1" y2="20.32" width="0" layer="19" extent="1-1"/>
-<wire x1="67.31" y1="13.97" x2="38.1" y2="20.32" width="0" layer="19" extent="1-1"/>
+<via x="35.56" y="16.51" extent="1-16" drill="0.6"/>
+<via x="38.1" y="11.43" extent="1-16" drill="0.6"/>
+<wire x1="38.1" y1="11.43" x2="35.56" y2="16.51" width="0.254" layer="16"/>
+<via x="69.85" y="6.985" extent="1-16" drill="0.6"/>
+<via x="69.85" y="4.445" extent="1-16" drill="0.6"/>
+<wire x1="69.85" y1="4.445" x2="69.85" y2="6.985" width="0.254" layer="16"/>
 </signal>
 <signal name="GND">

Commit message: Add missing wires
Connections:
- new net !RFSH: IC1.28
- net !INT: now also IC1.16
- net !NMI: now also IC1.17
- net !RESET: now also IC1.26
- net !WAIT: now also IC1.24
Changed lines of the file:
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@@
 <?xml version="1.0" encoding="utf-8"?>
 <!DOCTYPE eagle SYSTEM "eagle.dtd">
-<eagle version="8.0.0">
+<eagle version="8.2.2">
 <drawing>
 <settings>
@@
 <elements>
 <element name="IC1" library="zilog" package="DIL40" value="Z80CPU" x="66.04" y="21.59">
+<attribute name="MF" value="" x="66.04" y="21.59" size="1.778" layer="27" display="off"/>
+<attribute name="MPN" value="" x="66.04" y="21.59" size="1.778" layer="27" display="off"/>
 <attribute name="OC_FARNELL" value="unknown" x="66.04" y="21.59" size="1.778" layer="27" display="off"/>
-<attribute name="MPN" value="" x="66.04" y="21.59" size="1.778" layer="27" display="off"/>
-<attribute name="MF" value="" x="66.04" y="21.59" size="1.778" layer="27" display="off"/>
 </element>
 <element name="JP1" library="jean" package="2X25/90" value="" x="72.39" y="0" rot="R180"/>
 <element name="QG1" library="crystal" package="DIL14S" value="6 MHz" x="20.955" y="23.495" smashed="yes">
+<attribute name="MF" value="" x="20.955" y="23.495" size="1.778" layer="27" display="off"/>
+<attribute name="MPN" value="" x="20.955" y="23.495" size="1.778" layer="27" display="off"/>
+<attribute name="NAME" x="31.115" y="29.0576" size="1.27" layer="25" ratio="10"/>
 <attribute name="OC_FARNELL" value="unknown" x="20.955" y="23.495" size="1.778" layer="27" display="off"/>
 <attribute name="OC_NEWARK" value="unknown" x="20.955" y="23.495" size="1.778" layer="27" display="off"/>
-<attribute name="MPN" value="" x="20.955" y="23.495" size="1.778" layer="27" display="off"/>
-<attribute name="MF" value="" x="20.955" y="23.495" size="1.778" layer="27" display="off"/>
-<attribute name="NAME" x="31.115" y="29.0576" size="1.27" layer="25" ratio="10"/>
 <attribute name="VALUE" x="13.335" y="22.6822" size="1.27" layer="27" ratio="10"/>
 </element>
@@
 <wire x1="0.69" y1="11.43" x2="2.54" y2="11.43" width="0.254" layer="1"/>
 <wire x1="0.6858" y1="11.43" x2="0.69" y2="11.43" width="0.254" layer="1"/>
+<contactref element="IC1" pad="26"/>
+<wire x1="77.28" y1="29.21" x2="77.47" y2="29.21" width="0" layer="19" extent="1-1"/>
 </signal>
 <signal name="!WAIT">
@@
 <wire x1="20.3454" y1="8.6868" x2="20.32" y2="8.89" width="0.254" layer="1"/>
 <wire x1="20.3454" y1="6.4008" x2="20.32" y2="6.35" width="0.254" layer="1"/>
+<contactref element="IC1" pad="24"/>
+<wire x1="20.32" y1="8.89" x2="82.55" y2="29.21" width="0" layer="19" extent="1-1"/>
 </signal>
 <signal name="!MREQ">
@@
 <wire x1="5.0292" y1="8.6868" x2="5.08" y2="8.89" width="0.254" layer="1"/>
 <wire x1="5.0292" y1="8.6868" x2="5.06" y2="8.6868" width="0.254" layer="1"/>
+<contactref element="IC1" pad="17"/>
+<wire x1="5.08" y1="8.89" x2="82.55" y2="13.97" width="0" layer="19" extent="1-1"/>
 </signal>
 <signal name="!INT">
@@
 <wire x1="10.287" y1="8.6868" x2="10.16" y2="8.89" width="0.254" layer="1"/>
 <wire x1="10.287" y1="6.4008" x2="10.16" y2="6.35" width="0.254" layer="1"/>
+<contactref element="IC1" pad="16"/>
+<wire x1="10.287" y1="8.6868" x2="80.01" y2="13.97" width="0" layer="19" extent="1-1"/>
 </signal>
 <signal name="!BUSAK">
@@
 <wire x1="54.6354" y1="14.1732" x2="54.61" y2="13.97" width="0.254" layer="16"/>
 </signal>
+<signal name="!RFSH">
+<contactref element="IC1" pad="28"/>
+</signal>
 </signals>
