File: Memory.brd (EAGLE design)
At the start: 106.7 x 54.3 mm, 14 parts, among them IC1 AT28C256ZIF, IC2 HM62256DIP, IC3 74LS139N, IC4 HM62256DIP

Commit message: Fix Routing Issues with PowerPlanes
Routing:
- net GND: track 0.00 -> 14.6 mm, vias 0 -> 8
- net VCC: track 0.00 -> 9.52 mm, vias 0 -> 6
- net N$6: track 119.3 -> 120.1 mm
Changed lines of the file:
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@@
 <contactref element="V2" pad="16"/>
 <contactref element="V1" pad="14"/>
-<wire x1="80.01" y1="48.26" x2="88.9" y2="41.91" width="0" layer="19" extent="1-1"/>
-<wire x1="92.71" y1="30.48" x2="88.9" y2="41.91" width="0" layer="19" extent="1-1"/>
-<wire x1="69.85" y1="24.13" x2="69.85" y2="36.83" width="0" layer="19" extent="1-1"/>
+<via x="90.805" y="41.275" extent="1-16" drill="0.6"/>
+<via x="90.17" y="39.37" extent="1-16" drill="0.6"/>
+<wire x1="90.17" y1="39.37" x2="90.805" y2="39.37" width="0.4064" layer="16"/>
+<wire x1="90.805" y1="39.37" x2="90.805" y2="41.275" width="0.4064" layer="16"/>
+<via x="87.63" y="43.18" extent="1-16" drill="0.6"/>
+<via x="83.82" y="42.545" extent="1-16" drill="0.6"/>
+<wire x1="83.82" y1="42.545" x2="87.63" y2="42.545" width="0.4064" layer="1"/>
+<wire x1="87.63" y1="42.545" x2="87.63" y2="43.18" width="0.4064" layer="1"/>
+<via x="74.93" y="12.7" extent="1-16" drill="0.6"/>
+<via x="77.47" y="12.7" extent="1-16" drill="0.6"/>
+<wire x1="74.93" y1="12.7" x2="77.47" y2="12.7" width="0.4064" layer="16"/>
 </signal>
 <signal name="GND">
@@
 <contactref element="V2" pad="8"/>
 <contactref element="V1" pad="7"/>
-<wire x1="87.63" y1="29.21" x2="87.63" y2="16.51" width="0" layer="19" extent="1-1"/>
-<wire x1="92.71" y1="35.56" x2="87.63" y2="29.21" width="0" layer="19" extent="1-1"/>
-<wire x1="69.85" y1="16.51" x2="68.58" y2="3.81" width="0" layer="19" extent="1-1"/>
-<wire x1="39.37" y1="46.99" x2="17.78" y2="46.99" width="0" layer="19" extent="1-1"/>
+<via x="74.295" y="11.43" extent="1-16" drill="0.6"/>
+<wire x1="74.295" y1="11.43" x2="73.025" y2="11.43" width="0.4064" layer="1"/>
+<wire x1="73.025" y1="11.43" x2="73.025" y2="13.97" width="0.4064" layer="1"/>
+<via x="73.025" y="13.97" extent="1-16" drill="0.6"/>
+<via x="96.52" y="48.26" extent="1-16" drill="0.6"/>
+<via x="100.33" y="48.26" extent="1-16" drill="0.6"/>
+<wire x1="96.52" y1="48.26" x2="100.33" y2="48.26" width="0.4064" layer="1"/>
+<via x="89.535" y="25.4" extent="1-16" drill="0.6"/>
+<via x="89.535" y="21.59" extent="1-16" drill="0.6"/>
+<wire x1="89.535" y1="21.59" x2="89.535" y2="25.4" width="0.4064" layer="1"/>
+<via x="29.845" y="50.165" extent="1-16" drill="0.6"/>
+<via x="29.845" y="46.99" extent="1-16" drill="0.6"/>
+<wire x1="29.845" y1="46.99" x2="29.845" y2="50.165" width="0.254" layer="1"/>
 </signal>
 <signal name="!MREQ">
@@
 <wire x1="15" y1="31.5" x2="4" y2="20.5" width="0.254" layer="1"/>
 <wire x1="15" y1="47.5" x2="15" y2="31.5" width="0.254" layer="1"/>
-<wire x1="17.5" y1="50" x2="15" y2="47.5" width="0.254" layer="1"/>
-<wire x1="55" y1="50" x2="17.5" y2="50" width="0.254" layer="1"/>
+<wire x1="15" y1="47.5" x2="17.5" y2="50" width="0.254" layer="1"/>
 <wire x1="55.5" y1="50.5" x2="55" y2="50" width="0.254" layer="16"/>
 <wire x1="71.5" y1="50.5" x2="55.5" y2="50.5" width="0.254" layer="16"/>
@@
 <wire x1="72.5" y1="48.5" x2="72.39" y2="48.26" width="0.254" layer="16"/>
 <via x="55" y="50" extent="1-16" drill="0.6096"/>
+<wire x1="17.5" y1="50" x2="19.05" y2="51.435" width="0.254" layer="1"/>
+<wire x1="19.05" y1="51.435" x2="48.26" y2="51.435" width="0.254" layer="1"/>
+<wire x1="48.26" y1="51.435" x2="52.07" y2="50.165" width="0.254" layer="1"/>
+<wire x1="52.07" y1="50.165" x2="55" y2="50" width="0.254" layer="1"/>
 </signal>
 <signal name="N$9">

Commit message: Add pullup
Connections:
- net GND: no longer V2.6
- net VCC: now also V2.6
Changed lines of the file:
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@@
 <via x="77.47" y="12.7" extent="1-16" drill="0.6"/>
 <wire x1="74.93" y1="12.7" x2="77.47" y2="12.7" width="0.4064" layer="16"/>
+<contactref element="V2" pad="6"/>
 </signal>
 <signal name="GND">
@@
 <contactref element="IC4" pad="14"/>
 <contactref element="C4" pad="2"/>
-<contactref element="V2" pad="6"/>
 <contactref element="C5" pad="2"/>
 <contactref element="C6" pad="2"/>
